File: tactictoe-pcb.kicad_sch (KiCad schematic)
At the start: 86 parts, among them J1 USB_C_Receptacle_USB2.0_16P, J2 Conn_01x04, T1 Touchpad, T2 Touchpad, T3 Touchpad, T4 Touchpad, T5 Touchpad, T6 Touchpad, T7 Touchpad, T8 Touchpad, T9 Touchpad, U1 F042G6U6TR, U2 TLV74033PDBVR

Commit message: major v2 changes
Parts:
- removed D1, D2, D3, D4, D5: SK6805-EC15, tictactoe-bolt-footprints:SK6805-EC15, symbol tictactoe:SK6805-EC15
- removed R1, R2, R3: 10k, Resistor_SMD:R_0603_1608Metric_Pad0.98x0.95mm_HandSolder, symbol Device:R
- removed TP1: NRST, TestPoint:TestPoint_Pad_D1.0mm, symbol Connector:TestPoint
- removed TP2: PF0, TestPoint:TestPoint_Pad_D1.0mm, symbol Connector:TestPoint
- removed TP3: PF1, TestPoint:TestPoint_Pad_D1.0mm, symbol Connector:TestPoint
- removed TP4: PB8, TestPoint:TestPoint_Pad_D1.0mm, symbol Connector:TestPoint
- removed TP5: PA15, TestPoint:TestPoint_Pad_D1.0mm, symbol Connector:TestPoint
- added D1, D2, D3, D4, D5: XL-1615RGBC, tactictoe-footprints:XL-1615RGBC-WS2812B-S, symbol tactictoe:XL-1615RGBC-WS2812B-S
- C1, C2, C3, C4, C5, C6, C7, C8, C9: footprint Capacitor_SMD:C_0603_1608Metric_Pad1.08x0.95mm_HandSolder -> Capacitor_SMD:C_0603_1608Metric
- D10, D11, D12, D13, D14, D15, D16, D17, D18, D19, D20, D21, D22, D23, D24, D25, D26, D27, D28, D29, D30, D31, D32, D33, D34, D35, D36, D37, D38, D39, D40, D41, D42, D43, D44, D45, D6, D7, D8, D9: value SK6805-EC15 -> XL-1615RGBC; footprint tictactoe-bolt-footprints:SK6805-EC15 -> tactictoe-footprints:XL-1615RGBC-WS2812B-S; symbol tictactoe:SK6805-EC15 -> tactictoe:XL-1615RGBC-WS2812B-S
- J1: footprint tictactoe-bolt-footprints:USB_C_Receptacle_TYPE-C-16P-CB1-6-073 -> tactictoe-footprints:USB_C_Receptacle_TYPE-C-16P-CB1-6-073
- J2: footprint Connector_PinHeader_2.54mm:PinHeader_1x04_P2.54mm_Vertical -> tactictoe-footprints:tactictoe-sw-pins
- R10, R11, R12, R13, R14, R4, R5, R6, R7, R8, R9: footprint Resistor_SMD:R_0603_1608Metric_Pad0.98x0.95mm_HandSolder -> Resistor_SMD:R_0603_1608Metric
- T1, T2, T3, T4, T5, T6, T7, T8, T9: footprint tictactoe-bolt-footprints:Touch-pad -> tactictoe-footprints:Touch-pad_XL-1615; symbol tictactoe:Touchpad -> tactictoe:Touchpad
Connections:
- net +5V: now also D10.3 (VDD), D11.3 (VDD), D12.3 (VDD), D13.3 (VDD), D14.3 (VDD), D15.3 (VDD), D16.3 (VDD), D17.3 (VDD), D18.3 (VDD), D19.3 (VDD), D20.3 (VDD), D21.3 (VDD), D22.3 (VDD), D23.3 (VDD), D24.3 (VDD), D25.3 (VDD), D26.3 (VDD), D27.3 (VDD), D28.3 (VDD), D29.3 (VDD), D30.3 (VDD), D31.3 (VDD), D32.3 (VDD), D33.3 (VDD), D34.3 (VDD), D35.3 (VDD), D36.3 (VDD), D37.3 (VDD), D38.3 (VDD), D39.3 (VDD), D40.3 (VDD), D41.3 (VDD), D42.3 (VDD), D43.3 (VDD), D44.3 (VDD), D45.3 (VDD), D6.3 (VDD), D7.3 (VDD), D8.3 (VDD), D9.3 (VDD), J2.4 (Pin_4), D1.3 (VDD), D2.3 (VDD), D3.3 (VDD), D4.3 (VDD), D5.3 (VDD); no longer D10.2 (VDD), D11.2 (VDD), D12.2 (VDD), D13.2 (VDD), D14.2 (VDD), D15.2 (VDD), D16.2 (VDD), D17.2 (VDD), D18.2 (VDD), D19.2 (VDD), D20.2 (VDD), D21.2 (VDD), D22.2 (VDD), D23.2 (VDD), D24.2 (VDD), D25.2 (VDD), D26.2 (VDD), D27.2 (VDD), D28.2 (VDD), D29.2 (VDD), D30.2 (VDD), D31.2 (VDD), D32.2 (VDD), D33.2 (VDD), D34.2 (VDD), D35.2 (VDD), D36.2 (VDD), D37.2 (VDD), D38.2 (VDD), D39.2 (VDD), D40.2 (VDD), D41.2 (VDD), D42.2 (VDD), D43.2 (VDD), D44.2 (VDD), D45.2 (VDD), D6.2 (VDD), D7.2 (VDD), D8.2 (VDD), D9.2 (VDD), J2.1 (Pin_1)
- net GND: now also D10.1 (VSS), D11.1 (VSS), D12.1 (VSS), D13.1 (VSS), D14.1 (VSS), D15.1 (VSS), D16.1 (VSS), D17.1 (VSS), D18.1 (VSS), D19.1 (VSS), D20.1 (VSS), D21.1 (VSS), D22.1 (VSS), D23.1 (VSS), D24.1 (VSS), D25.1 (VSS), D26.1 (VSS), D27.1 (VSS), D28.1 (VSS), D29.1 (VSS), D30.1 (VSS), D31.1 (VSS), D32.1 (VSS), D33.1 (VSS), D34.1 (VSS), D35.1 (VSS), D36.1 (VSS), D37.1 (VSS), D38.1 (VSS), D39.1 (VSS), D40.1 (VSS), D41.1 (VSS), D42.1 (VSS), D43.1 (VSS), D44.1 (VSS), D45.1 (VSS), D6.1 (VSS), D7.1 (VSS), D8.1 (VSS), D9.1 (VSS), J2.1 (Pin_1), D1.1 (VSS), D2.1 (VSS), D3.1 (VSS), D4.1 (VSS), D5.1 (VSS); no longer D10.4 (VSS), D11.4 (VSS), D12.4 (VSS), D13.4 (VSS), D14.4 (VSS), D15.4 (VSS), D16.4 (VSS), D17.4 (VSS), D18.4 (VSS), D19.4 (VSS), D20.4 (VSS), D21.4 (VSS), D22.4 (VSS), D23.4 (VSS), D24.4 (VSS), D25.4 (VSS), D26.4 (VSS), D27.4 (VSS), D28.4 (VSS), D29.4 (VSS), D30.4 (VSS), D31.4 (VSS), D32.4 (VSS), D33.4 (VSS), D34.4 (VSS), D35.4 (VSS), D36.4 (VSS), D37.4 (VSS), D38.4 (VSS), D39.4 (VSS), D40.4 (VSS), D41.4 (VSS), D42.4 (VSS), D43.4 (VSS), D44.4 (VSS), D45.4 (VSS), D6.4 (VSS), D7.4 (VSS), D8.4 (VSS), D9.4 (VSS), J2.4 (Pin_4)
- net LED_CH2: no longer names the net of U1.26 (PB5)
- net LED_CH2: no longer D31.1 (DIN)
- net LED_CH3 renamed LED_T3C3
- net LED_T3C3: now also D16.2 (DIN); no longer D16.1 (DIN)
- net LED_CH4 renamed LED_T3C4
- net LED_T3C4: now also D1.2 (DIN)
- net PA15: no longer names the net of U1.23 (PA15)
- net PB8 renamed LED_T16C1
- net LED_T16C1: now also D31.2 (DIN)
- net PF0: no longer names the net of U1.2 (PF0)
- net PF1: no longer names the net of U1.3 (PF1)
- removed net USB_D+: J1.A6 (D+), J1.B6 (D+), U1.20 (PA10/PA12)
- removed net USB_D-: J1.A7 (D-), J1.B7 (D-), U1.19 (PA9/PA11)
- new net: D36.4 (DOUT), D37.2 (DIN)
- new net: D37.4 (DOUT), D38.2 (DIN)
- new net: D20.4 (DOUT), D21.2 (DIN)
- new net: D21.4 (DOUT), D22.2 (DIN)
- new net: D10.2 (DIN), D9.4 (DOUT)
- new net: D10.4 (DOUT), D11.2 (DIN)
- new net: D7.4 (DOUT), D8.2 (DIN)
- new net: D8.4 (DOUT), D9.2 (DIN)
- new net: D1.4 (DOUT), D2.2 (DIN)
- new net: D14.4 (DOUT), D15.2 (DIN)
- new net: D3.4 (DOUT), D4.2 (DIN)
- new net: D4.4 (DOUT), D5.2 (DIN)
- new net: D13.4 (DOUT), D14.2 (DIN)
- new net: D11.4 (DOUT), D12.2 (DIN)
- new net: D12.4 (DOUT), D13.2 (DIN)
- new net: D16.4 (DOUT), D17.2 (DIN)
- new net: D31.4 (DOUT), D32.2 (DIN)
- new net: D2.4 (DOUT), D3.2 (DIN)
- new net: D42.4 (DOUT), D43.2 (DIN)
- new net: D43.4 (DOUT), D44.2 (DIN)
- new net: D38.4 (DOUT), D39.2 (DIN)
- new net: D39.4 (DOUT), D40.2 (DIN)
- new net: D5.4 (DOUT), D6.2 (DIN)
- new net: D6.4 (DOUT), D7.2 (DIN)
- new net: D18.4 (DOUT), D19.2 (DIN)
- new net: D19.4 (DOUT), D20.2 (DIN)
- new net: D33.4 (DOUT), D34.2 (DIN)
- new net: D34.4 (DOUT), D35.2 (DIN)
- new net: D23.4 (DOUT), D24.2 (DIN)
- new net: D24.4 (DOUT), D25.2 (DIN)
- new net: D29.4 (DOUT), D30.2 (DIN)
- new net: D17.4 (DOUT), D18.2 (DIN)
- new net: D25.4 (DOUT), D26.2 (DIN)
- new net: D26.4 (DOUT), D27.2 (DIN)
- new net: D44.4 (DOUT), D45.2 (DIN)
- new net: D22.4 (DOUT), D23.2 (DIN)
- new net: D32.4 (DOUT), D33.2 (DIN)
- new net: D40.4 (DOUT), D41.2 (DIN)
- new net: D35.4 (DOUT), D36.2 (DIN)
- new net: D41.4 (DOUT), D42.2 (DIN)
- new net: D28.4 (DOUT), D29.2 (DIN)
- new net: D27.4 (DOUT), D28.2 (DIN)
- no-connect marks 5 -> 15
Other:
- note added: "RGB LED: XL-1615RGBC-WS2812B-S"
- moved on the sheet: J2, R4, R5
